File: Logic Circuits 2/BasicGates2.brd (EAGLE design)
At the start: 100 x 100 mm, 34 parts, among them T1 2N3904, T2 2N3904, T3 2N3904, T4 2N3904, T5 2N3904, T6 2N3904, T7 2N3904, T8 2N3904

Commit message: Update board. Upload AND/OR
Signed-off-by: William Woody <woody@alumni.caltech.edu>
Parts:
- removed 1: LED, led:LED5MM
- removed R4: 330, resistor:0309/10
- removed SW1: (no value), special:EDG-01
- moved R19 70.1 mm to (22.9, 12.7)
- moved T8 69.3 mm to (34.3, 12.7)
- moved R17 68.3 mm to (22.9, 21.6)
- moved T6 67.4 mm to (34.3, 21.6)
- moved R15 66.5 mm to (10.2, 20.3)
- moved R18 66.5 mm to (6.35, 20.3)
- moved SW3 66.5 mm to (8.89, 33.0)
- moved R16 65.6 mm to (33.0, 33.0)
- moved R1 58.5 mm to (55.9, 33.0)
- moved R13 53.4 mm to (62.2, 20.3), turned to 270 degrees
- moved R14 53.4 mm to (62.2, 33.0)
- moved 3 52.8 mm to (69.8, 33.0)
- moved T7 52.8 mm to (69.8, 20.3)
- moved J1 50.8 mm to (66.0, 5.08)
- moved T2 45.9 mm to (55.9, 21.6)
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Connections:
- removed net N$121: 1.A, R4.1
- removed net N$124: 1.K, T2.1
- net GND: no longer R1.1
- net N$1: now also R6.1; no longer R3.1
- net N$16: now also R3.1; no longer R13.1
- net N$3: now also R1.1, R13.1, T2.1; no longer R1.2, R5.1, SW1.1
- net N$7: now also R5.1; no longer R6.1
- net VCC: now also R1.2; no longer R4.2, SW1.2
Routing:
- net GND: track 219.1 -> 263.7 mm
- net N$121: track 12.0 -> 0.00 mm
- net VCC: track 215.5 -> 205.2 mm
- net N$124: track 8.89 -> 0.00 mm
- net N$19: track 10.1 -> 3.18 mm
- net N$3: track 16.3 -> 11.4 mm
- net N$12: track 18.4 -> 22.5 mm
- net N$16: track 22.8 -> 26.5 mm
- net N$1: track 15.0 -> 11.4 mm
- net N$21: track 19.4 -> 22.5 mm
- net N$18: track 10.2 -> 13.0 mm
- net N$10: track 3.81 -> 6.35 mm
- net N$20: track 5.87 -> 7.67 mm
- net N$17: track 5.87 -> 7.67 mm
- net N$9: track 11.4 -> 13.0 mm
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Other:
- board text added: "AND Gate"
- board text added: "AND and OR Gate Both are made by adding a NOT gate to a NAND and a NOR gate."
- board text added: "Logic Table: 0 0 -> 0 0 1 -> 0 1 0 -> 0 1 1 -> 1"
- board text added: "Logic Table: 0 0 -> 0 0 1 -> 1 1 0 -> 1 1 1 -> 1"
- board text added: "OR Gate"
- board text removed: "Basic Digital Gates using NPN transistors. This card shows three basic gates: the NOT gate, the NAND gate, and the NOR gate. The difference between a NAND gate and a NOR gate is how the transistors are wired: on the NAND gate, they are wired in sequence, while on a NOR gate, they are wired in parallel."
- board text removed: "Logic Table: 0 -> 1 1 -> 0"
- board text removed: "Logic Table: 0 0 -> 1 0 1 -> 0 1 0 -> 0 1 1 -> 0"
- board text removed: "Logic Table: 0 0 -> 1 0 1 -> 1 1 0 -> 1 1 1 -> 0"
